Commit message: 添加moveit配置

File: src/arm_description/urdf/arm.urdf (robot description, URDF)
Before this commit: robot arm_description, 10 links, 9 joints
Joints:
- joint camera_arm_joint: origin xyz=0.0630000000000002 0 0 rpy=0 0 0 -> xyz=0.0380000000000002 0 0 rpy=0 0 0
- joint fork_joint_L: origin xyz=0.0645000000000001 -0.0544327264438395 0 rpy=0 0 0 -> xyz=0.039500000000001 -0.0544327264438395 0 rpy=0 0 0
- joint fork_joint_R: origin xyz=0.0645000000000003 0.0544327264438282 0 rpy=0 0 0 -> xyz=0.0395000000000003 0.0544327264438282 0 rpy=0 0 0
