Commit message: arm,desk,pallet解耦，第一次规划成功

File: src/arm_description/urdf/all.urdf.xacro (robot description, xacro)
@@ -6,8 +6,8 @@
     <xacro:desk />
     <!-- <xacro:pallet /> -->
-    <joint name="block_arm_joint" type="fixed">
+    <!-- <joint name="block_arm_joint" type="fixed">
     <origin xyz="0 0 0.07" rpy="0 0 0"/>
     <parent link="bolck_link"/>
     <child link="base_link"/>
-    </joint>
+    </joint> -->
 </robot>

File: src/arm_description/urdf/arm.urdf.xacro (robot description, xacro)
@@ -3,5 +3,5 @@
      Commit Version: 1.6.0-4-g7f85cfe  Build Version: 1.6.7995.38578
      For more information, please see http://wiki.ros.org/sw_urdf_exporter -->
-<robot xmlns:xacro="http://www.ros.org/wiki/xacro">
+<robot name="arm_description" xmlns:xacro="http://www.ros.org/wiki/xacro">
   <xacro:include filename="$(find arm_description)/urdf/arm_description.ros2_control.xacro" />
   <link

File: src/moveit_config/config/arm_description.urdf.xacro (robot description, xacro)
@@ -3,7 +3,7 @@
     <xacro:arg name="initial_positions_file" default="initial_positions.yaml" />
     <!-- Import arm_description urdf file -->
-    <xacro:include filename="$(find arm_description)/urdf/arm.urdf" />
+    <xacro:include filename="$(find arm_description)/urdf/arm.urdf.xacro" />
     <!-- Import control_xacro -->
-    <xacro:include filename="arm_description.ros2_control.xacro" />
-    <xacro:arm_description_ros2_control name="FakeSystem" initial_positions_file="$(arg initial_positions_file)"/>
+    <!-- <xacro:include filename="arm_description.ros2_control.xacro" /> -->
+    <!-- <xacro:arm_description_ros2_control name="FakeSystem" initial_positions_file="$(arg initial_positions_file)"/> -->
 </robot>
