Commit message: 调整机械臂模型

File: src/arm_description/urdf/arm.urdf.xacro (robot description, xacro)
@@ -10,5 +10,5 @@
     <link name="world" />
     <joint name="gazebo_world_joint" type="fixed">
-      <origin xyz="-0.25 0.19 0.275" rpy="0 0 0" />
+      <origin xyz="-0.25 0.1 0.275" rpy="0 0 0" />
       <parent link="world" />
       <child link="base_link" />
@@ -59,15 +59,15 @@
     <inertial>
       <origin
-        xyz="2.844E-09 -0.0018983 0.088853"
-        rpy="0 0 0" />
-      <mass
-        value="0.96068" />
-      <inertia
-        ixx="0.0026125"
-        ixy="-5.235E-10"
-        ixz="-2.5725E-10"
-        iyy="0.002564"
-        iyz="0.00011151"
-        izz="0.0003434" />
+        xyz="1.3529E-07 0.00018621 0.085433"
+        rpy="0 0 0" />
+      <mass
+        value="0.90979" />
+      <inertia
+        ixx="0.0023552"
+        ixy="-7.2006E-11"
+        ixz="-6.7195E-09"
+        iyy="0.0023529"
+        iyz="-1.0941E-05"
+        izz="0.00028703" />
     </inertial>
     <visual>
@@ -100,5 +100,5 @@
     <origin
       xyz="0 0 0.01"
-      rpy="0 0 3.1415926" />
+      rpy="0 0 0" />
     <parent
       link="base_link" />
@@ -108,6 +108,6 @@
       xyz="0 0 1" />
     <limit
-      lower="-1.5708"
-      upper="1.5708"
+      lower="-1.57"
+      upper="1.57"
       effort="50"
       velocity="1.5" />
@@ -117,15 +117,15 @@
     <inertial>
       <origin
-        xyz="3.99321170061077E-07 0.00243945434428174 0.10000016404977"
-        rpy="0 0 0" />
-      <mass
-        value="1.49514311129629" />
-      <inertia
-        ixx="0.0092672086833684"
-        ixy="-3.45316524239455E-08"
-        ixz="2.128280625616E-08"
-        iyy="0.00917221220256816"
-        iyz="-8.41134008902218E-09"
-        izz="0.000552274337038071" />
+        xyz="-0.12356 -0.0039664 0.008897"
+        rpy="0 0 0" />
+      <mass
+        value="1.7751" />
+      <inertia
+        ixx="0.00085052"
+        ixy="-0.00032685"
+        ixz="0.0010043"
+        iyy="0.014556"
+        iyz="2.3539E-05"
+        izz="0.014725" />
     </inertial>
     <visual>
@@ -140,5 +140,5 @@
         name="">
         <color
-          rgba="0.898039215686275 0.917647058823529 0.929411764705882 1" />
+          rgba="0.89804 0.91765 0.92941 1" />
       </material>
     </visual>
@@ -157,6 +157,6 @@
     type="revolute">
     <origin
-      xyz="0 -0.08 0.15"
-      rpy="0 1.0 0" />
+      xyz="0 0.065 0.15"
+      rpy="0 0 0" />
     <parent
       link="shoulder_link" />
@@ -164,8 +164,8 @@
       link="arm_link_1" />
     <axis
-      xyz="0 1 0" />
+      xyz="0 -1 0" />
     <limit
-      lower="-2.6179938"
-      upper="1.1"
+      lower="-3.14"
+      upper="0.3"
       effort="50"
       velocity="1.5" />
@@ -175,15 +175,15 @@
     <inertial>
       <origin
-        xyz="1.84935938307083E-07 -0.00142742297622724 0.0811160068194484"
-        rpy="0 0 0" />
-      <mass
-        value="1.27771981813338" />
-      <inertia
-        ixx="0.00602979199459265"
-        ixy="1.99665710014809E-09"
-        ixz="3.61991807814648E-09"
-        iyy="0.00598043834668597"
-        iyz="-0.000147930160932861"
-        izz="0.000443651831504686" />
+        xyz="0.069958 0.0038771 0.032231"
+        rpy="0 0 0" />
+      <mass
+        value="1.3456" />
+      <inertia
+        ixx="0.0016571"
+        ixy="0.00036495"
+        ixz="-0.0022841"
+        iyy="0.006418"
+        iyz="0.00016813"
+        izz="0.0055625" />
     </inertial>
     <visual>
@@ -198,5 +198,5 @@
         name="">
         <color
-          rgba="0.898039215686275 0.917647058823529 0.929411764705882 1" />
+          rgba="0.89804 0.91765 0.92941 1" />
       </material>
     </visual>
@@ -215,6 +215,6 @@
     type="revolute">
     <origin
-      xyz="0 0.08 0.2"
-      rpy="0 -2.5 0" />
+      xyz="-0.22941 -0.12 0.016519"
+      rpy="0 0 0" />
     <parent
       link="arm_link_1" />
@@ -222,8 +222,8 @@
       link="arm_link_2" />
     <axis
-      xyz="0 1 0" />
+      xyz="0 -1 0" />
     <limit
-      lower="-0.1"
-      upper="2.8179938"
+      lower="-1.1"
+      upper="3.14"
       effort="50"
       velocity="1.5" />
@@ -233,15 +233,15 @@
     <inertial>
       <origin
-        xyz="0.00484427832761932 -1.19442283489963E-08 0.0299999925216045"
-        rpy="0 0 0" />
-      <mass
-        value="0.376466363968247" />
-      <inertia
-        ixx="0.00015732940102775"
-        ixy="2.42567535480483E-10"
-        ixz="9.20593423415752E-11"
-        iyy="0.00020045101820395"
-        iyz="1.04465083118944E-10"
-        izz="0.00015578083797655" />
+        xyz="0.027247 -0.0048443 0.012553"
+        rpy="0 0 0" />
+      <mass
+        value="0.37647" />
+      <inertia
+        ixx="0.0001636"
+        ixy="-1.8511E-10"
+        ixz="-1.6977E-05"
+        iyy="0.00015733"
+        iyz="1.8179E-10"
+        izz="0.00019263" />
     </inertial>
     <visual>
@@ -256,5 +256,5 @@
         name="">
         <color
-          rgba="0.898039215686275 0.917647058823529 0.929411764705882 1" />
+          rgba="0.89804 0.91765 0.92941 1" />
       </material>
     </visual>
@@ -273,6 +273,6 @@
     type="revolute">
     <origin
-      xyz="0 0 0.2"
-      rpy="0 0 -3.1415926" />
+      xyz="0.18165 0 0.083688"
+      rpy="0 0 0" />
     <parent
       link="arm_link_2" />
@@ -280,8 +280,8 @@
       link="wrist_link_1" />
     <axis
-      xyz="0 0 1" />
+      xyz="0.90824 0 0.41844" />
     <limit
-      lower="-1.6"
-      upper="1.6"
+      lower="-2.1"
+      upper="2.1"
       effort="50"
       velocity="1.5" />
@@ -291,15 +291,15 @@
     <inertial>
       <origin
-        xyz="-0.025 0.00476010124384936 -5.3487070328373E-10"
-        rpy="0 0 0" />
-      <mass
-        value="0.213833773430547" />
-      <inertia
-        ixx="5.90471340191189E-05"
-        ixy="-3.62696963816373E-20"
-        ixz="5.85438282709314E-12"
-        iyy="6.19132185170091E-05"
-        iyz="1.83189050496876E-12"
-        izz="7.58889080283275E-05" />
+        xyz="0.0047601 0.025 -5.3504E-10"
+        rpy="0 0 0" />
+      <mass
+        value="0.21383" />
+      <inertia
+        ixx="6.1913E-05"
+        ixy="-5.4902E-21"
+        ixz="1.8319E-12"
+        iyy="5.9047E-05"
+        iyz="-5.8544E-12"
+        izz="7.5889E-05" />
     </inertial>
     <visual>
@@ -314,5 +314,5 @@
         name="">
         <color
-          rgba="0.176470588235294 1 0.529411764705882 1" />
+          rgba="0.17647 1 0.52941 1" />
       </material>
     </visual>
@@ -331,81 +331,81 @@
     type="revolute">
     <origin
-      xyz="0.09 0 0.03"
-      rpy="0.2 0 0" />
+      xyz="0.027247 -0.09 0.012553"
+      rpy="0 0 0" />
     <parent
       link="wrist_link_1" />
     <child
       link="wrist_link_2" />
+    <axis
+      xyz="0 -1 0" />
+    <limit
+      lower="-2.1"
+      upper="2.1"
+      effort="50"
+      velocity="1.5" />
+  </joint>
+  <link
+    name="wrist_link_3">
+    <inertial>
+      <origin
+        xyz="0.039939 -1.1351E-13 -1.7214E-13"
+        rpy="0 0 0" />
+      <mass
+        value="0.28823" />
+      <inertia
+        ixx="0.00024443"
+        ixy="1.3258E-19"
+        ixz="1.023E-20"
+        iyy="0.00016365"
+        iyz="7.1532E-20"
+        izz="0.00034072" />
+    </inertial>
+    <visual>
+      <origin
+        xyz="0 0 0"
+        rpy="0 0 0" />
+      <geometry>
+        <mesh
+          filename="package://arm_description/meshes/arm/wrist_link_3.STL" />
+      </geometry>
+      <material
+        name="">
+        <color
+          rgba="1 0.27059 0.73333 1" />
+      </material>
+    </visual>
+    <collision>
+      <origin
+        xyz="0 0 0"
+        rpy="0 0 0" />
+      <geometry>
+        <mesh
+          filename="package://arm_description/meshes/arm/wrist_link_3.STL" />
+      </geometry>
+    </collision>
+  </link>
+  <joint
+    name="wrist_joint_23"
+    type="revolute">
+    <origin
+      xyz="0.03 0.025 0"
+      rpy="0 0 0" />
+    <parent
+      link="wrist_link_2" />
+    <child
+      link="wrist_link_3" />
     <axis
       xyz="1 0 0" />
     <limit
-      lower="-1.0"
-      upper="1.0"
+      lower="-2.1"
+      upper="2.1"
       effort="50"
       velocity="1.5" />
   </joint>
   <link
-    name="wrist_link_3">
-    <inertial>
-      <origin
-        xyz="0.0379528150536633 -0.00306208343475713 1.84945643244561E-08"
-        rpy="0 0 0" />
-      <mass
-        value="0.332413101297219" />
-      <inertia
-        ixx="0.000271281133244879"
-        ixy="-1.31842072075757E-05"
-        ixz="-4.53971642475216E-12"
-        iyy="0.000181807242336193"
-        iyz="-7.12639945244701E-12"
-        izz="0.000374581320728992" />
-    </inertial>
-    <visual>
-      <origin
-        xyz="-0.025 0 0"
-        rpy="0 0 0" />
-      <geometry>
-        <mesh
-          filename="package://arm_description/meshes/arm/wrist_link_3.STL" />
-      </geometry>
-      <material
-        name="">
-        <color
-          rgba="1 0.270588235294118 0.733333333333333 1" />
-      </material>
-    </visual>
-    <collision>
-      <origin
-        xyz="-0.025 0 0"
-        rpy="0 0 0" />
-      <geometry>
-        <mesh
-          filename="package://arm_description/meshes/arm/wrist_link_3.STL" />
-      </geometry>
-    </collision>
-  </link>
-  <joint
-    name="wrist_joint_23"
-    type="revolute">
-    <origin
-      xyz="-0.025 0.06 0"
-      rpy="0 -1.57 0" />
-    <parent
-      link="wrist_link_2" />
-    <child
-      link="wrist_link_3" />
-    <axis
-      xyz="0 1 0" />
-    <limit
-      lower="-2.6179938"
-      upper="2.6179938"
-      effort="50"
-      velocity="1.5" />
-  </joint>
-  <link
     name="camera_arm_link">
     <inertial>
       <origin
-        xyz="0.00017826 0 0"
+        xyz="0.00017826 4.5935E-15 -1.3661E-13"
         rpy="0 0 0" />
       <mass
@@ -413,8 +413,8 @@
       <inertia
         ixx="6.6534E-07"
-        ixy="-7.307E-23"
-        ixz="8.7818E-23"
+        ixy="-1.0694E-22"
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
File: src/arm_description/urdf/desk.gazebo.urdf.xacro (robot description, xacro)
@@ -24,3 +24,15 @@
     <material>Gazebo/Grey</material>
   </gazebo>
+  <gazebo reference="s_1_L">
+    <material>Gazebo/Blue</material>
+  </gazebo>
+  <gazebo reference="s_2_L">
+    <material>Gazebo/Blue</material>
+  </gazebo>
+  <gazebo reference="s_3_L">
+    <material>Gazebo/Blue</material>
+  </gazebo>
+  <gazebo reference="s_4_L">
+    <material>Gazebo/Blue</material>
+  </gazebo>
 </robot>

File: src/arm_description/urdf/desk.urdf.xacro (robot description, xacro)
@@ -9,15 +9,15 @@
       <inertial>
         <origin
-          xyz="0.2633 -1.3648E-06 0.41758"
-          rpy="0 0 0" />
-        <mass
-          value="175.57" />
-        <inertia
-          ixx="15.115"
-          ixy="0.00035798"
-          ixz="0.18408"
-          iyy="15.317"
-          iyz="-3.2904E-05"
-          izz="11.622" />
+          xyz="0.26330028162089 4.70495183503534E-05 0.41757762572946"
+          rpy="0 0 0" />
+        <mass
+          value="175.56800657568" />
+        <inertia
+          ixx="15.1168947961039"
+          ixy="0.00340084138859789"
+          ixz="0.184078944732021"
+          iyy="15.3169560302271"
+          iyz="-0.000325921549303988"
+          izz="11.6240723783388" />
       </inertial>
       <visual>
@@ -32,5 +32,5 @@
           name="">
           <color
-            rgba="0.79216 0.81961 0.93333 1" />
+            rgba="0.792156862745098 0.819607843137255 0.933333333333333 1" />
         </material>
       </visual>
@@ -49,14 +49,14 @@
       <inertial>
         <origin
-          xyz="2.7756E-17 0 0.001"
+          xyz="2.77555756156289E-17 0 0.00100000000000006"
           rpy="0 0 0" />
         <mass
           value="0.0162" />
         <inertia
-          ixx="1.094E-05"
-          ixy="1.6756E-21"
-          ixz="-6.3137E-38"
-          iyy="1.094E-05"
-          iyz="-4.191E-24"
+          ixx="1.09404E-05"
+          ixy="1.67558837898401E-21"
+          ixz="-6.3136903608619E-38"
+          iyy="1.09404E-05"
+          iyz="-4.19104843693536E-24"
           izz="2.187E-05" />
       </inertial>
@@ -72,5 +72,5 @@
           name="">
           <color
-            rgba="0.92549 0.92549 0.92549 1" />
+            rgba="0.925490196078431 0.925490196078431 0.925490196078431 1" />
         </material>
       </visual>
@@ -102,14 +102,14 @@
       <inertial>
         <origin
-          xyz="-2.7756E-17 -2.7756E-17 0.001"
+          xyz="-2.77555756156289E-17 -2.77555756156289E-17 0.00100000000000006"
           rpy="0 0 0" />
         <mass
           value="0.0162" />
         <inertia
-          ixx="1.094E-05"
-          ixy="5.1772E-22"
-          ixz="9.9262E-24"
-          iyy="1.094E-05"
-          iyz="2.9779E-23"
+          ixx="1.09404E-05"
+          ixy="5.17717379383552E-22"
+          ixz="9.92616735063634E-24"
+          iyy="1.09404E-05"
+          iyz="2.9778502051909E-23"
           izz="2.187E-05" />
       </inertial>
@@ -125,5 +125,5 @@
           name="">
           <color
-            rgba="0.92549 0.92549 0.92549 1" />
+            rgba="0.925490196078431 0.925490196078431 0.925490196078431 1" />
         </material>
       </visual>
@@ -208,5 +208,5 @@
       <inertial>
         <origin
-          xyz="0 -2.77555756156289E-17 0.001"
+          xyz="-2.77555756156289E-17 -2.77555756156289E-17 0.001"
           rpy="0 0 0" />
         <mass
@@ -264,12 +264,12 @@
           rpy="0 0 0" />
         <mass
-          value="0.7" />
-        <inertia
-          ixx="0.00086917"
-          ixy="8.4279E-20"
-          ixz="1.4167E-21"
-          iyy="0.00086917"
-          iyz="5.1428E-36"
-          izz="0.0011667" />
+          value="0.700000000000001" />
+        <inertia
+          ixx="0.000869166666666668"
+          ixy="-6.39679281766446E-21"
+          ixz="3.10876902924011E-20"
+          iyy="0.000869166666666668"
+          iyz="-1.65303893084384E-36"
+          izz="0.00116666666666667" />
       </inertial>
       <visual>
@@ -284,5 +284,5 @@
           name="">
           <color
-            rgba="0.79216 0.81961 0.93333 1" />
+            rgba="0.792156862745098 0.819607843137255 0.933333333333333 1" />
         </material>
       </visual>
@@ -301,5 +301,5 @@
       type="fixed">
       <origin
-        xyz="-0.25 0.0199999999999995 0.00499999999999999"
+        xyz="-0.25 0.19 0.005"
         rpy="0 0 0" />
       <parent
@@ -307,4 +307,216 @@
       <child
         link="bolck_link" />
+      <axis
+        xyz="0 0 0" />
+    </joint>
+    <link
+      name="s_1_L">
+      <inertial>
+        <origin
+          xyz="0.0061913 0.001 -0.00013874"
+          rpy="0 0 0" />
+        <mass
+          value="0.0053851" />
+        <inertia
+          ixx="3.8704E-06"
+          ixy="-2.0456E-21"
+          ixz="-2.3702E-07"
+          iyy="4.362E-06"
+          iyz="-8.4608E-22"
+          izz="4.9511E-07" />
+      </inertial>
+      <visual>
+        <origin
+          xyz="0 0 0"
+          rpy="0 0 0" />
+        <geometry>
+          <mesh
+            filename="package://arm_description/meshes/desk/s_1_L.STL" />
+        </geometry>
+        <material
+          name="">
+          <color
+            rgba="0.97647 1 0.29412 1" />
+        </material>
+      </visual>
+      <collision>
+        <origin
+          xyz="0 0 0"
+          rpy="0 0 0" />
+        <geometry>
+          <mesh
+            filename="package://arm_description/meshes/desk/s_1_L.STL" />
+        </geometry>
+      </collision>
+    </link>
+    <joint
+      name="s_1_J"
+      type="fixed">
+      <origin
+        xyz="0.40942 0.17674 0.65022"
+        rpy="0 0 1.5708" />
+      <parent
+        link="desk_link" />
+      <child
+        link="s_1_L" />
+      <axis
+        xyz="0 0 0" />
+    </joint>
+    <link
+      name="s_2_L">
+      <inertial>
+        <origin
+          xyz="-2.7756E-17 0.0025 0"
+          rpy="0 0 0" />
+        <mass
+          value="0.022" />
+        <inertia
+          ixx="2.1579E-05"
+          ixy="-2.5789E-20"
+          ixz="1.6E-06"
+          iyy="2.8667E-05"
+          iyz="5.062E-21"
+          izz="7.1792E-06" />
+      </inertial>
+      <visual>
+        <origin
+          xyz="0 0 0"
+          rpy="0 0 0" />
+        <geometry>
+          <mesh
+            filename="package://arm_description/meshes/desk/s_2_L.STL" />
+        </geometry>
+        <material
+          name="">
+          <color
+            rgba="0.97647 1 0.29412 1" />
+        </material>
+      </visual>
+      <collision>
+        <origin
+          xyz="0 0 0"
+          rpy="0 0 0" />
+        <geometry>
+          <mesh
+            filename="package://arm_description/meshes/desk/s_2_L.STL" />
+        </geometry>
+      </collision>
+    </link>
+    <joint
+      name="s_2_J"
+      type="fixed">
+      <origin
+        xyz="0.40942 -0.19 0.65"
+        rpy="0 0 1.5708" />
+      <parent
+        link="desk_link" />
+      <child
+        link="s_2_L" />
+      <axis
+        xyz="0 0 0" />
+    </joint>
+    <link
+      name="s_3_L">
+      <inertial>
+        <origin
+          xyz="-0.0036364 0.0025 0"
+          rpy="0 0 0" />
+        <mass
+          value="0.022" />
+        <inertia
+          ixx="2.1579E-05"
+          ixy="-2.4788E-20"
+          ixz="-2.3193E-21"
+          iyy="2.8376E-05"
+          iyz="-2.4423E-22"
+          izz="6.8883E-06" />
+      </inertial>
+      <visual>
+        <origin
+          xyz="0 0 0"
+          rpy="0 0 0" />
+        <geometry>
+          <mesh
+            filename="package://arm_description/meshes/desk/s_3_L.STL" />
+        </geometry>
+        <material
+          name="">
+          <color
+            rgba="0.97647 1 0.29412 1" />
+        </material>
+      </visual>
+      <collision>
+        <origin
+          xyz="0 0 0"
+          rpy="0 0 0" />
+        <geometry>
+          <mesh
+            filename="package://arm_description/meshes/desk/s_3_L.STL" />
+        </geometry>
+      </collision>
+    </link>
+    <joint
+      name="s_3_J"
+      type="fixed">
+      <origin
+        xyz="0.40942 0.19 0.25"
+        rpy="0 0 1.5708" />
+      <parent
+        link="desk_link" />
+      <child
+        link="s_3_L" />
+      <axis
+        xyz="0 0 0" />
+    </joint>
+    <link
+      name="s_4_L">
+      <inertial>
+        <origin
+          xyz="0.0055937 0.0025 0.0073044"
+          rpy="0 0 0" />
+        <mass
+          value="0.010984" />
+        <inertia
+          ixx="5.1745E-06"
+          ixy="-6.3019E-21"
+          ixz="2.0561E-07"
+          iyy="7.0614E-06"
+          iyz="7.693E-22"
+          izz="1.9327E-06" />
+      </inertial>
+      <visual>
+        <origin
+          xyz="0 0 0"
+          rpy="0 0 0" />
+        <geometry>
+          <mesh
+            filename="package://arm_description/meshes/desk/s_4_L.STL" />
+        </geometry>
+        <material
+          name="">
+          <color
+            rgba="0.97647 1 0.29412 1" />
+        </material>
+      </visual>
+      <collision>
+        <origin
+          xyz="0 0 0"
+          rpy="0 0 0" />
+        <geometry>
+          <mesh
+            filename="package://arm_description/meshes/desk/s_4_L.STL" />
+        </geometry>
+      </collision>
+    </link>
+    <joint
+      name="s_4_J"
+      type="fixed">
+      <origin
+        xyz="0.40942 -0.20085 0.235"
+        rpy="0 0 1.5708" />
+      <parent
+        link="desk_link" />
+      <child
+        link="s_4_L" />
       <axis
         xyz="0 0 0" />

Commit message: 添加叉齿附着

File: src/arm_description/urdf/arm.urdf.xacro (robot description, xacro)
@@ -4,8 +4,9 @@
      For more information, please see http://wiki.ros.org/sw_urdf_exporter -->
 <robot name="arm_description" xmlns:xacro="http://www.ros.org/wiki/xacro">
-  <xacro:arg name="use_gazebo" default="true" />
+  <xacro:arg name="use_gazebo" default="false" />
+  <xacro:arg name="include_world_joint" default="true" />
   <xacro:include filename="$(find arm_description)/urdf/arm_description.ros2_control.xacro" />
-  <!-- Anchor the simulated arm while keeping the normal MoveIt model unchanged. -->
-  <xacro:if value="$(arg use_gazebo)">
+  <!-- Use the same fixed base transform in Gazebo, MoveIt, and robot_state_publisher. -->
+  <xacro:if value="$(arg include_world_joint)">
     <link name="world" />
     <joint name="gazebo_world_joint" type="fixed">
@@ -640,7 +641,19 @@
     <gazebo reference="fork_link_L">
       <material>Gazebo/Orange</material>
+      <mu1>1.0</mu1>
+      <mu2>1.0</mu2>
+      <kp>1000000.0</kp>
+      <kd>100.0</kd>
+      <minDepth>0.001</minDepth>
+      <maxVel>0.01</maxVel>
     </gazebo>
     <gazebo reference="fork_link_R">
       <material>Gazebo/Orange</material>
+      <mu1>1.0</mu1>
+      <mu2>1.0</mu2>
+      <kp>1000000.0</kp>
+      <kd>100.0</kd>
+      <minDepth>0.001</minDepth>
+      <maxVel>0.01</maxVel>
     </gazebo>
   </xacro:if>

File: src/arm_description/urdf/pallet.gazebo.urdf.xacro (robot description, xacro)
@@ -8,5 +8,11 @@
   </gazebo>
   <gazebo reference="pallet_link">
-  <material>Gazebo/Grey</material>
+    <material>Gazebo/Grey</material>
+    <mu1>1.0</mu1>
+    <mu2>1.0</mu2>
+    <kp>1000000.0</kp>
+    <kd>100.0</kd>
+    <minDepth>0.001</minDepth>
+    <maxVel>0.01</maxVel>
   </gazebo>
   <gazebo reference="target_f_link">
